Commit message: Updating editor.launch.py for more controls -play pause -speed -remove waypoints from view -slider

File: src/arm_description/urdf/camera_arm.urdf (robot description, URDF)
Before this commit: robot camera_arm, 8 links, 7 joints
Joints:
- joint pillar_joint: origin xyz=0.22 0.35 0.2 rpy=0 0 0 -> xyz=0.50 7.00 0.2 rpy=0 0 0

File: src/arm_description_v2/urdf/camera_arm_v2.urdf (robot description, URDF)
Before this commit: robot camera_arm_v2, 6 links, 5 joints
Links:
- added link camera_optical_frame
- added link pillar; visual box size=0.05 0.05 0.4
Joints:
- added joint camera_optical_joint: type fixed, parent Pitch_Gimbal, child camera_optical_frame, origin xyz=-0.06147775915604879 -0.05799207543869661 -0.11446999999999949 rpy=-1.5465200834087727 1.5707963267948966 2.380470733578473
- added joint pillar_joint: type fixed, parent base_link, child pillar, origin xyz=0 0.6 0.2 rpy=0 0 0
- joint Pitch: origin xyz=-0.000599768 -0.0618564 0.114769 rpy=0 0 -0.7854 -> xyz=-0.000761782 -0.0579922 0.114769 rpy=0 0 -0.785398163397449
- joint R: origin xyz=0.0943 0.06275 0.027475 rpy=-1.5708 1.4816 -1.5708 -> xyz=0.0943 0.06275 0.027475 rpy=-1.5707963267949 1.48162448210916 -1.5707963267949
- joint Theta: origin xyz=0 0 0 rpy=-1.5708 0 -1.5708 -> xyz=0 0 0 rpy=-1.5707963267949 0 -1.5707963267949
- joint Yaw: origin xyz=0.063543 0.0433336 -0.444201 rpy=-3.1416 0 -1.4816 -> xyz=0.063543 0.0433336 -0.444201 rpy=-3.14159265358979 0 -1.48162448210916
- joint Z: origin xyz=0.10025 -0.30653 0.3248 rpy=1.5708 -1.5708 0 -> xyz=0.10025 -0.30653 0.3248 rpy=1.5707963267949 -1.5707963267949 0
