Commit message: Moving the camera point to inside the camera instead of on the lens for more accuracy

File: src/arm_description_v2/urdf/camera_arm_v2.urdf (robot description, URDF)
Before this commit: robot camera_arm_v2, 8 links, 7 joints
Links:
- removed link pillar
Joints:
- removed joint pillar_joint
- joint camera_optical_joint: origin xyz=-0.06147775915604879 -0.05799207543869661 -0.11446999999999949 rpy=-1.5465200834087727 1.5707963267948966 2.380470733578473 -> xyz=-0.010721351559766147 -0.00723566784241355 -0.11446999999999949 rpy=-1.5465200834087727 1.5707963267948966 2.380470733578473

Commit message: Add speed/timing, tangent arcs and S-curve to camera paths

File: src/arm_description_v2/urdf/camera_arm_v2.urdf (robot description, URDF)
Before this commit: robot camera_arm_v2, 7 links, 6 joints
Joints:
- joint Pitch: type revolute -> continuous
- joint Theta: type revolute -> continuous
- joint Yaw: type revolute -> continuous
